File: mm_external_uart.kicad_sch (KiCad schematic)
At the start: 0 parts

Commit message: TP3
Parts:
- added J4: Conn_01x04, Connector_PinHeader_2.54mm:PinHeader_1x04_P2.54mm_Vertical, symbol Connector_Generic:Conn_01x04
- added R18: 100, Resistor_SMD:R_0603_1608Metric, symbol Device:R
Connections:
- new net: J4.3 (Pin_3), R18.2
- new net +BATT: J4.2 (Pin_2)
- new net EXT_UART_RX: J4.4 (Pin_4)
- new net EXT_UART_TX: R18.1
- new net GND: J4.1 (Pin_1)
Changed lines of the file:
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@@
 (kicad_sch (version 20230121) (generator eeschema)
   (paper "A4")
+  (junction (at 149.86 91.44) (diameter 0) (color 0 0 0 0)
+  )
+  (wire (pts (xy 151.13 91.44) (xy 149.86 91.44))
+    (stroke (width 0) (type default))
+  )
+  (wire (pts (xy 149.86 93.98) (xy 142.24 93.98))
+    (stroke (width 0) (type default))
+  )
+  (wire (pts (xy 140.97 91.44) (xy 140.97 109.22))
+    (stroke (width 0) (type default))
+  )
+  (wire (pts (xy 149.86 91.44) (xy 140.97 91.44))
+    (stroke (width 0) (type default))
+  )
+  (wire (pts (xy 116.84 99.06) (xy 149.86 99.06))
+    (stroke (width 0) (type default))
+  )
+  (wire (pts (xy 137.16 96.52) (xy 149.86 96.52))
+    (stroke (width 0) (type default))
+  )
+  (wire (pts (xy 142.24 93.98) (xy 142.24 82.55))
+    (stroke (width 0) (type default))
+  )
+  (wire (pts (xy 116.84 96.52) (xy 129.54 96.52))
+    (stroke (width 0) (type default))
+  )
+  (hierarchical_label "EXT_UART_TX" (shape output) (at 116.84 96.52 180) (fields_autoplaced)
+    (effects (font (size 1.27 1.27)) (justify right))
+  )
+  (hierarchical_label "EXT_UART_RX" (shape input) (at 116.84 99.06 180) (fields_autoplaced)
+    (effects (font (size 1.27 1.27)) (justify right))
+  )
+  (symbol (lib_id "Connector_Generic:Conn_01x04") (at 154.94 93.98 0) (unit 1)
+    (in_bom yes) (on_board yes) (dnp no) (fields_autoplaced)
+    (property "Reference" "J4" (at 157.48 93.98 0)
+      (effects (font (size 1.27 1.27)) (justify left))
+    )
+    (property "Value" "Conn_01x04" (at 157.48 96.52 0)
+      (effects (font (size 1.27 1.27)) (justify left))
+    )
+    (property "Footprint" "Connector_PinHeader_2.54mm:PinHeader_1x04_P2.54mm_Vertical" (at 154.94 93.98 0)
+      (effects (font (size 1.27 1.27)) hide)
+    )
+    (property "Datasheet" "~" (at 154.94 93.98 0)
+      (effects (font (size 1.27 1.27)) hide)
+    )
+    (pin "4")
+    (pin "1")
+    (pin "3")
+    (pin "2")
+    (instances
+      (project "minimouse"
+        (path "/d8fa4cba-2469-4231-847f-065b6b829f44/d17bb1c7-f68a-465e-9a17-5858ef86fc30"
+          (reference "J4") (unit 1)
+        )
+      )
+    )
+  )
+  (symbol (lib_id "Device:R") (at 133.35 96.52 90) (unit 1)
+    (in_bom yes) (on_board yes) (dnp no) (fields_autoplaced)
+    (property "Reference" "R18" (at 133.35 90.17 90)
+      (effects (font (size 1 1)))
+    )
+    (property "Value" "100" (at 133.35 92.71 90)
+      (effects (font (size 1 1)))
+    )
+    (property "Footprint" "Resistor_SMD:R_0603_1608Metric" (at 133.35 98.298 90)
+      (effects (font (size 1.27 1.27)) hide)
+    )
+    (property "Datasheet" "~" (at 133.35 96.52 0)
+      (effects (font (size 1.27 1.27)) hide)
+    )
+    (pin "2")
+    (pin "1")
+    (instances
+      (project "minimouse"
+        (path "/d8fa4cba-2469-4231-847f-065b6b829f44/d17bb1c7-f68a-465e-9a17-5858ef86fc30"
+          (reference "R18") (unit 1)
+        )
+      )
+    )
+  )
+  (symbol (lib_id "power:+BATT") (at 142.24 82.55 0) (unit 1)
+    (in_bom yes) (on_board yes) (dnp no) (fields_autoplaced)
+    (property "Reference" "#PWR026" (at 142.24 86.36 0)
+      (effects (font (size 1.27 1.27)) hide)
+    )
+    (property "Value" "+BATT" (at 142.24 77.47 0)
+      (effects (font (size 1.27 1.27)))
+    )
+    (property "Footprint" "" (at 142.24 82.55 0)
+      (effects (font (size 1.27 1.27)) hide)
+    )
+    (property "Datasheet" "" (at 142.24 82.55 0)
+      (effects (font (size 1.27 1.27)) hide)
+    )
+    (pin "1")
+    (instances
+      (project "minimouse"
+        (path "/d8fa4cba-2469-4231-847f-065b6b829f44/d17bb1c7-f68a-465e-9a17-5858ef86fc30"
+          (reference "#PWR026") (unit 1)
+        )
+      )
+    )
+  )
+  (symbol (lib_id "power:GND") (at 140.97 109.22 0) (unit 1)
+    (in_bom yes) (on_board yes) (dnp no) (fields_autoplaced)
+    (property "Reference" "#PWR027" (at 140.97 115.57 0)
+      (effects (font (size 1.27 1.27)) hide)
+    )
+    (property "Value" "GND" (at 140.97 114.3 0)
+      (effects (font (size 1.27 1.27)))
+    )
+    (property "Footprint" "" (at 140.97 109.22 0)
+      (effects (font (size 1.27 1.27)) hide)
+    )
+    (property "Datasheet" "" (at 140.97 109.22 0)
+      (effects (font (size 1.27 1.27)) hide)
+    )
+    (pin "1")
+    (instances
+      (project "minimouse"
+        (path "/d8fa4cba-2469-4231-847f-065b6b829f44/d17bb1c7-f68a-465e-9a17-5858ef86fc30"
+          (reference "#PWR027") (unit 1)
+        )
+      )
+    )
+  )
 )
