File: mm_motor_control.kicad_sch (KiCad schematic)
At the start: 0 parts

Commit message: fin tp2
Parts:
- added C9: C, symbol Device:C
- added CEN: 10nF, symbol Device:C
- added CRCOFF: 22nF, symbol Device:C
- added CSPOL: 22uF, symbol Device:C
- added Cs: 2.2uF, symbol Device:C
- added R10, R11: 10k, symbol Device:R
- added R12: R, symbol Device:R
- added REN: 18k, symbol Device:R
- added ROFF: 47k, symbol Device:R
- added RRCOFF: 1k, symbol Device:R
- added RSNSA, RSNSB: 330m, symbol Device:R
- added U3: STSPIN240, Package_DFN_QFN:VQFN-16-1EP_3x3mm_P0.5mm_EP1.8x1.8mm, symbol Driver_Motor:STSPIN240
Connections:
- net EN: now also REN.2
- net FAULT: now also CEN.1, REN.1, U3.13 (EN/FLT)
- net OUT_A1: now also U3.3 (OUTA1)
- net OUT_A2: now also U3.5 (OUTA2)
- net OUT_B1: now also U3.10 (OUTB1)
- net OUT_B2: now also U3.8 (OUTB2)
- net PHASE_A: now also U3.1 (PHA)
- net PHASE_B: now also U3.15 (PHB)
- net PWM_A: now also U3.2 (PWMA)
- net PWM_B: now also U3.16 (PWMB)
- net STBY/RESET: now also C9.1, R12.2, U3.14 (STBY/RESET)
- new net: ROFF.1, RRCOFF.1, U3.12 (TOFF)
- new net: CRCOFF.1, RRCOFF.2
- new net: R10.1, R11.2, U3.11 (REF)
- new net: RSNSA.1, U3.4 (SENSEA)
- new net: RSNSB.1, U3.9 (SENSEB)
- new net +BATT: R11.1
- new net GND: CEN.2, CRCOFF.2, CSPOL.2, Cs.2, R10.2, ROFF.2, RSNSB.2, U3.17 (EPAD), U3.7 (GND)
- new net VDD: R12.1
- new net VS: CSPOL.1, Cs.1, U3.6 (VS)

Commit message: TP3
Parts:
- C9: footprint (none) -> Capacitor_SMD:C_0603_1608Metric
- CEN1: renamed from CEN; footprint (none) -> Capacitor_SMD:C_0603_1608Metric
- CRCOFF1: renamed from CRCOFF; footprint (none) -> Capacitor_SMD:C_0603_1608Metric
- CSPOL1: renamed from CSPOL; footprint (none) -> Capacitor_SMD:C_0603_1608Metric
- Cs1: renamed from Cs; footprint (none) -> Capacitor_SMD:C_0603_1608Metric
- R10, R11, R12: footprint (none) -> Resistor_SMD:R_0603_1608Metric
- REN1: renamed from REN; footprint (none) -> Resistor_SMD:R_0603_1608Metric
- ROFF1: renamed from ROFF; footprint (none) -> Resistor_SMD:R_0603_1608Metric
- RRCOFF1: renamed from RRCOFF; footprint (none) -> Resistor_SMD:R_0603_1608Metric
- RSNSA1: renamed from RSNSA; footprint (none) -> Resistor_SMD:R_2512_6332Metric
- RSNSB1: renamed from RSNSB; footprint (none) -> Resistor_SMD:R_2512_6332Metric
Changed lines of the file:
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@@
   (symbol (lib_id "Device:R") (at 130.81 110.49 0) (unit 1)
     (in_bom yes) (on_board yes) (dnp no) (fields_autoplaced)
-    (property "Reference" "ROFF" (at 133.35 109.22 0)
+    (property "Reference" "ROFF1" (at 133.35 109.22 0)
       (effects (font (size 1.27 1.27)) (justify left))
     )
@@
       (effects (font (size 1.27 1.27)) (justify left))
     )
-    (property "Footprint" "" (at 129.032 110.49 90)
+    (property "Footprint" "Resistor_SMD:R_0603_1608Metric" (at 129.032 110.49 90)
       (effects (font (size 1.27 1.27)) hide)
     )
@@
       (project "minimouse"
         (path "/d8fa4cba-2469-4231-847f-065b6b829f44/0999fad3-9a14-4ede-b729-a71c3dbbdf8e"
-          (reference "ROFF") (unit 1)
+          (reference "ROFF1") (unit 1)
         )
       )
@@
   (symbol (lib_id "Device:R") (at 120.65 105.41 0) (unit 1)
     (in_bom yes) (on_board yes) (dnp no) (fields_autoplaced)
-    (property "Reference" "RRCOFF" (at 123.19 104.14 0)
+    (property "Reference" "RRCOFF1" (at 123.19 104.14 0)
       (effects (font (size 1.27 1.27)) (justify left))
     )
@@
       (effects (font (size 1.27 1.27)) (justify left))
     )
-    (property "Footprint" "" (at 118.872 105.41 90)
+    (property "Footprint" "Resistor_SMD:R_0603_1608Metric" (at 118.872 105.41 90)
       (effects (font (size 1.27 1.27)) hide)
     )
@@
       (project "minimouse"
         (path "/d8fa4cba-2469-4231-847f-065b6b829f44/0999fad3-9a14-4ede-b729-a71c3dbbdf8e"
-          (reference "RRCOFF") (unit 1)
+          (reference "RRCOFF1") (unit 1)
         )
       )
@@
   (symbol (lib_id "Device:C") (at 193.04 59.69 0) (unit 1)
     (in_bom yes) (on_board yes) (dnp no) (fields_autoplaced)
-    (property "Reference" "Cs" (at 196.85 58.42 0)
+    (property "Reference" "Cs1" (at 196.85 58.42 0)
       (effects (font (size 1.27 1.27)) (justify left))
     )
@@
       (effects (font (size 1.27 1.27)) (justify left))
     )
-    (property "Footprint" "" (at 194.0052 63.5 0)
+    (property "Footprint" "Capacitor_SMD:C_0603_1608Metric" (at 194.0052 63.5 0)
       (effects (font (size 1.27 1.27)) hide)
     )
@@
       (project "minimouse"
         (path "/d8fa4cba-2469-4231-847f-065b6b829f44/0999fad3-9a14-4ede-b729-a71c3dbbdf8e"
-          (reference "Cs") (unit 1)
+          (reference "Cs1") (unit 1)
         )
       )
@@
   (symbol (lib_id "Device:C") (at 204.47 59.69 0) (unit 1)
     (in_bom yes) (on_board yes) (dnp no) (fields_autoplaced)
-    (property "Reference" "CSPOL" (at 208.28 58.42 0)
+    (property "Reference" "CSPOL1" (at 208.28 58.42 0)
       (effects (font (size 1.27 1.27)) (justify left))
     )
@@
       (effects (font (size 1.27 1.27)) (justify left))
     )
-    (property "Footprint" "" (at 205.4352 63.5 0)
+    (property "Footprint" "Capacitor_SMD:C_0603_1608Metric" (at 205.4352 63.5 0)
       (effects (font (size 1.27 1.27)) hide)
     )
@@
       (project "minimouse"
         (path "/d8fa4cba-2469-4231-847f-065b6b829f44/0999fad3-9a14-4ede-b729-a71c3dbbdf8e"
-          (reference "CSPOL") (unit 1)
+          (reference "CSPOL1") (unit 1)
         )
       )
@@
   (symbol (lib_id "Device:C") (at 120.65 114.3 0) (unit 1)
     (in_bom yes) (on_board yes) (dnp no)
-    (property "Reference" "CRCOFF" (at 121.92 110.49 0)
+    (property "Reference" "CRCOFF1" (at 121.92 110.49 0)
       (effects (font (size 1 1)) (justify left))
     )
@@
       (effects (font (size 1 1)) (justify left))
     )
-    (property "Footprint" "" (at 121.6152 118.11 0)
+    (property "Footprint" "Capacitor_SMD:C_0603_1608Metric" (at 121.6152 118.11 0)
       (effects (font (size 1.27 1.27)) hide)
     )
@@
       (project "minimouse"
         (path "/d8fa4cba-2469-4231-847f-065b6b829f44/0999fad3-9a14-4ede-b729-a71c3dbbdf8e"
-          (reference "CRCOFF") (unit 1)
+          (reference "CRCOFF1") (unit 1)
         )
       )
@@
   (symbol (lib_id "Device:C") (at 77.47 96.52 0) (unit 1)
     (in_bom yes) (on_board yes) (dnp no) (fields_autoplaced)
-    (property "Reference" "CEN" (at 81.28 95.25 0)
+    (property "Reference" "CEN1" (at 81.28 95.25 0)
       (effects (font (size 1.27 1.27)) (justify left))
     )
@@
       (effects (font (size 1.27 1.27)) (justify left))
     )
-    (property "Footprint" "" (at 78.4352 100.33 0)
+    (property "Footprint" "Capacitor_SMD:C_0603_1608Metric" (at 78.4352 100.33 0)
       (effects (font (size 1.27 1.27)) hide)
     )
@@
       (project "minimouse"
         (path "/d8fa4cba-2469-4231-847f-065b6b829f44/0999fad3-9a14-4ede-b729-a71c3dbbdf8e"
-          (reference "CEN") (unit 1)
+          (reference "CEN1") (unit 1)
         )
       )
@@
       (effects (font (size 1.27 1.27)) (justify left))
     )
-    (property "Footprint" "" (at 42.8752 132.08 0)
+    (property "Footprint" "Capacitor_SMD:C_0603_1608Metric" (at 42.8752 132.08 0)
       (effects (font (size 1.27 1.27)) hide)
     )
@@
   (symbol (lib_id "Device:R") (at 67.31 88.9 270) (unit 1)
     (in_bom yes) (on_board yes) (dnp no)
-    (property "Reference" "REN" (at 67.31 95.25 90)
+    (property "Reference" "REN1" (at 67.31 95.25 90)
       (effects (font (size 1.27 1.27)))
     )
@@
       (effects (font (size 1.27 1.27)))
     )
-    (property "Footprint" "" (at 67.31 87.122 90)
+    (property "Footprint" "Resistor_SMD:R_0603_1608Metric" (at 67.31 87.122 90)
       (effects (font (size 1.27 1.27)) hide)
     )
@@
       (project "minimouse"
         (path "/d8fa4cba-2469-4231-847f-065b6b829f44/0999fad3-9a14-4ede-b729-a71c3dbbdf8e"
-          (reference "REN") (unit 1)
+          (reference "REN1") (unit 1)
         )
       )
@@
   (symbol (lib_id "Device:R") (at 171.45 82.55 0) (unit 1)
     (in_bom yes) (on_board yes) (dnp no) (fields_autoplaced)
-    (property "Reference" "RSNSA" (at 173.99 81.28 0)
+    (property "Reference" "RSNSA1" (at 173.99 81.28 0)
       (effects (font (size 1.27 1.27)) (justify left))
     )
@@
       (effects (font (size 1.27 1.27)) (justify left))
     )
-    (property "Footprint" "" (at 169.672 82.55 90)
+    (property "Footprint" "Resistor_SMD:R_2512_6332Metric" (at 169.672 82.55 90)
       (effects (font (size 1.27 1.27)) hide)
     )
@@
       (project "minimouse"
         (path "/d8fa4cba-2469-4231-847f-065b6b829f44/0999fad3-9a14-4ede-b729-a71c3dbbdf8e"
-          (reference "RSNSA") (unit 1)
+          (reference "RSNSA1") (unit 1)
         )
       )
@@
       (effects (font (size 1.27 1.27)) (justify left))
     )
-    (property "Footprint" "" (at 103.632 107.95 90)
+    (property "Footprint" "Resistor_SMD:R_0603_1608Metric" (at 103.632 107.95 90)
       (effects (font (size 1.27 1.27)) hide)
     )
@@
   (symbol (lib_id "power:+BATT") (at 88.9 100.33 0) (unit 1)
     (in_bom yes) (on_board yes) (dnp no) (fields_autoplaced)
-    (property "Reference" "#PWR036" (at 88.9 104.14 0)
+    (property "Reference" "#PWR010" (at 88.9 104.14 0)
       (effects (font (size 1.27 1.27)) hide)
     )
@@
     (instances
       (project "minimouse"
-        (path "/d8fa4cba-2469-4231-847f-065b6b829f44/3f9b0845-5778-418c-a7a8-03da2392145e"
-          (reference "#PWR036") (unit 1)
-        )
         (path "/d8fa4cba-2469-4231-847f-065b6b829f44/0999fad3-9a14-4ede-b729-a71c3dbbdf8e"
           (reference "#PWR010") (unit 1)
@@
       (effects (font (size 1.27 1.27)) (justify left))
     )
-    (property "Footprint" "" (at 103.632 118.11 90)
+    (property "Footprint" "Resistor_SMD:R_0603_1608Metric" (at 103.632 118.11 90)
       (effects (font (size 1.27 1.27)) hide)
     )
@@
       (effects (font (size 1.27 1.27)) (justify left))
     )
-    (property "Footprint" "" (at 40.132 115.57 90)
+    (property "Footprint" "Resistor_SMD:R_0603_1608Metric" (at 40.132 115.57 90)
       (effects (font (size 1.27 1.27)) hide)
     )
@@
   (symbol (lib_id "Device:R") (at 170.18 99.06 0) (unit 1)
     (in_bom yes) (on_board yes) (dnp no) (fields_autoplaced)
-    (property "Reference" "RSNSB" (at 172.72 97.79 0)
+    (property "Reference" "RSNSB1" (at 172.72 97.79 0)
       (effects (font (size 1.27 1.27)) (justify left))
     )
@@
       (effects (font (size 1.27 1.27)) (justify left))
     )
-    (property "Footprint" "" (at 168.402 99.06 90)
+    (property "Footprint" "Resistor_SMD:R_2512_6332Metric" (at 168.402 99.06 90)
       (effects (font (size 1.27 1.27)) hide)
     )
@@
       (project "minimouse"
         (path "/d8fa4cba-2469-4231-847f-065b6b829f44/0999fad3-9a14-4ede-b729-a71c3dbbdf8e"
-          (reference "RSNSB") (unit 1)
-        )
-      )
+          (reference "RSNSB1") (unit 1)
+        )
+      )

Commit message: tp3p3
Parts:
- C9: value C -> 1nF
Connections:
- net GND: now also RSNSA1.2
Changed lines of the file:
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@@
+    (stroke (width 0) (type default))
+  )
+  (wire (pts (xy 214.63 86.36) (xy 214.63 104.14))
+    (stroke (width 0) (type default))
+  )
+  (wire (pts (xy 171.45 86.36) (xy 214.63 86.36))
     (stroke (width 0) (type default))
   )
@@
     )
   )
+  (symbol (lib_id "power:GND") (at 214.63 104.14 0) (unit 1)
+    (in_bom yes) (on_board yes) (dnp no) (fields_autoplaced)
+    (property "Reference" "#PWR032" (at 214.63 110.49 0)
+      (effects (font (size 1.27 1.27)) hide)
+    )
+    (property "Value" "GND" (at 214.63 109.22 0)
+      (effects (font (size 1.27 1.27)))
+    )
+    (property "Footprint" "" (at 214.63 104.14 0)
+      (effects (font (size 1.27 1.27)) hide)
+    )
+    (property "Datasheet" "" (at 214.63 104.14 0)
+      (effects (font (size 1.27 1.27)) hide)
+    )
+    (pin "1")
+    (instances
+      (project "minimouse"
+        (path "/d8fa4cba-2469-4231-847f-065b6b829f44/0999fad3-9a14-4ede-b729-a71c3dbbdf8e"
+          (reference "#PWR032") (unit 1)
+        )
+      )
+    )
+  )
   (symbol (lib_id "Device:C") (at 77.47 96.52 0) (unit 1)
     (in_bom yes) (on_board yes) (dnp no) (fields_autoplaced)
@@
       (effects (font (size 1.27 1.27)) (justify left))
     )
-    (property "Value" "C" (at 45.72 129.54 0)
-      (effects (font (size 1.27 1.27)) (justify left))
-    )
+    (property "Value" "1nF" (at 45.72 129.54 0)
+      (effects (font (size 1.27 1.27)) (justify left))
+    )
